File: KiCad/Regulador.kicad_sch (KiCad schematic)
At the start: 225 parts, among them Q1 BC556, Q10 BC556, Q11 BC556, Q12 IRFZ44N, Q13 2N7000, Q14 BC556, Q15 BC547, Q16 BC556, Q17 BC556, Q18 IRFZ44N, Q19 2N7000, Q2 BC556, Q20 IRFZ44N, Q21 PJFET, Q23 BC547, Q24 BC547, Q25 BC547, Q26 BC547, Q27 BC547, Q3 BC807, Q4 IRF7328, Q6 IRFZ44N, Q7 2N7000, Q8 PJFET, SW1 SW_SPDT, U1 CA3096, U10 ICL7660, U11 TL431LP, U2 CA3096, U3 CA3096, U4 LM324A, U5 TL431LP, U6 TL431LP, U7 LM339, U8 TL431LP, U9 LM393

Commit message: Add files via upload
Parts:
- added TP_OUT1, TP_VCC1: TestPoint, TestPoint:TestPoint_THTPad_D4.0mm_Drill2.0mm, symbol Connector:TestPoint
- C1, C14, C16, C17, C2, C22, C9: footprint Capacitor_THT:C_Rect_L7.2mm_W3.5mm_P5.00mm_FKS2_FKP2_MKS2_MKP2 -> Capacitor_THT:C_Rect_L7.2mm_W3.0mm_P5.00mm_FKS2_FKP2_MKS2_MKP2
- C10: footprint Capacitor_THT:C_Disc_D7.5mm_W2.5mm_P5.00mm -> Capacitor_THT:CP_Radial_Tantal_D5.0mm_P2.50mm
- C11, C13, C8: footprint Capacitor_THT:CP_Radial_Tantal_D6.0mm_P2.50mm -> Capacitor_THT:CP_Radial_Tantal_D4.5mm_P2.50mm
- C15: value 300n -> 330n; footprint Capacitor_THT:C_Rect_L7.0mm_W2.5mm_P5.00mm -> Capacitor_THT:C_Rect_L7.2mm_W4.5mm_P5.00mm_FKS2_FKP2_MKS2_MKP2
- C3: value 30n -> 33n
- C4: footprint Capacitor_THT:C_Rect_L9.0mm_W3.8mm_P7.50mm_MKT -> Capacitor_THT:C_Disc_D3.8mm_W2.6mm_P2.50mm
- C5: footprint Capacitor_THT:C_Disc_D3.0mm_W1.6mm_P2.50mm -> Capacitor_THT:C_Disc_D3.8mm_W2.6mm_P2.50mm
- C6: footprint Capacitor_THT:C_Rect_L7.0mm_W2.5mm_P5.00mm -> Library_Marcos:C_Rect_L7.0mm_W2.0mm_P4.00mm
- C7: value 4.3n -> 4.7n; footprint Capacitor_THT:C_Rect_L7.0mm_W2.5mm_P5.00mm -> Library_Marcos:C_Rect_L7.0mm_W2.0mm_P4.00mm
- D1, D10, D13, D14, D15, D19, D2, D21, D3, D8, D9: footprint Diode_THT:D_DO-41_SOD81_P7.62mm_Horizontal -> Diode_THT:D_DO-35_SOD27_P7.62mm_Horizontal
- D11, D12, D17, D18, D4, D5, D6, D7: value 1N5817 -> 1N5819; symbol Diode:1N5817 -> Diode:1N5819
- D20: value Q_SCR_AGK -> TYN612; symbol Device:Q_SCR_AGK -> Device:Q_SCR_KAG
- F1: footprint Fuse:Fuseholder_Clip-5x20mm_Littelfuse_520_Inline_P20.50x5.80mm_D1.30mm_Horizontal -> Fuse:Fuseholder_Clip-5x20mm_Littelfuse_445-030_Inline_P20.50x5.20mm_D1.30mm_Horizontal
- INPUT1, OUTPUT1: footprint TerminalBlock:TerminalBlock_bornier-2_P5.08mm -> Library_Marcos:TerminalBlock_P5.08mm
- Q1, Q10, Q11, Q14, Q16, Q17, Q2: value BC556 -> BC557
- Q21, Q8: value PJFET -> J175
- R24: value 14k -> 15k
- R30, R31, R70, R73, R79: value 3k -> 3.3k
- R40: value 12k -> 10k
- R42: value 560 -> 510
- R53: value 2 -> 1
- R62: value 36k -> 20k
- R66: value 102k -> 100k
- R71, R72: footprint Resistor_THT:R_Axial_DIN0207_L6.3mm_D2.5mm_P7.62mm_Horizontal -> Resistor_THT:R_Axial_DIN0204_L3.6mm_D1.6mm_P5.08mm_Horizontal
- R78: value 8.2k -> 7.5k
- R81: value 82k -> 68k
- R82: value 820 -> 680
- RV1, RV10, RV11, RV12, RV13, RV2, RV3, RV4, RV5, RV6, RV7, RV8, RV9: footprint Potentiometer_THT:Potentiometer_Bourns_3266Y_Vertical -> Potentiometer_THT:Potentiometer_Bourns_3296W_Vertical
- Rsns1: footprint Resistor_THT:R_Axial_DIN0207_L6.3mm_D2.5mm_P7.62mm_Horizontal -> Resistor_THT:R_Axial_DIN0516_L15.5mm_D5.0mm_P20.32mm_Horizontal
- SW1: footprint Button_Switch_THT:SW_Slide_SPDT_Straight_CK_OS102011MS2Q -> Library_Marcos:SWITCH1; symbol Switch:SW_SPDT -> Marcos_Lib:Switch; Height (none) -> 4.7; Manufacturer_Name (none) -> KNITTER-SWITCH; Manufacturer_Part_Number (none) -> MFP113D-RA
- U1, U2, U3: footprint Package_DIP:DIP-16_W7.62mm_Socket_LongPads -> Library_Marcos:DIP-16
- U4: footprint Package_DIP:DIP-14_W7.62mm_Socket_LongPads -> Library_Marcos:CERDIP-14
- U7: footprint Package_DIP:CERDIP-14_W7.62mm_SideBrazed_LongPads_Socket -> Library_Marcos:CERDIP-14
- U9: footprint Package_DIP:CERDIP-8_W7.62mm_SideBrazed_LongPads_Socket -> Library_Marcos:CERDIP-8
Connections:
- net GND: now also D20.1 (K), SW1.MH1, SW1.MH2; no longer D20.3 (K)
- net OUT: now also TP_OUT1.1
- net VCC: now also TP_VCC1.1
- net VDOBL: now also D20.2 (A); no longer D20.1 (A)
- net at C22.1, D19.2 (A), R106.2: now also D20.3 (G); no longer D20.2 (G)
- no-connect marks 19 -> 18
Other:
- note added: "VZENER 15V"
